File: electronics/board/board.sch (KiCad schematic (older format))
At the start: 21 parts

Commit message: Board update
Parts:
- added C?: 100n, symbol Device:C
- added C?: 1u, symbol Device:C
- added C?: 100nF, symbol Device:C
- added D?: DIODE, symbol pspice:DIODE
- added F?: MSMF050 500mA, symbol Device:Polyfuse
- added F? (x2): CG0603MLC-05E, symbol Device:Polyfuse
- added J? (x16): Conn_01x02, symbol Connector_Generic:Conn_01x02
- added Q?: IRF7404, Package_SO:SOIC-8_3.9x4.9mm_P1.27mm, symbol Transistor_FET:IRF7404
- added R? (x2): 10K, symbol Device:R
- added R? (x2): 10k, symbol Device:R
- added U?: LMV358, symbol Amplifier_Operational:LMV358
Connections:
- net GND: now also C?.1, C?.2, F?.2, F?.2, R?.1; no longer U?.3 (DE), U?.30 (PB6)
- net at U?.10 (COM): now also J?.2 (Pin_2), J?.2 (Pin_2), J?.2 (Pin_2), J?.2 (Pin_2), J?.2 (Pin_2), J?.2 (Pin_2), J?.2 (Pin_2), J?.2 (Pin_2) (x2)
- net at U?.11 (O8): now also J?.1 (Pin_1) (x2)
- net at U?.12 (O7): now also J?.1 (Pin_1) (x2)
- net at U?.13 (O6): now also J?.1 (Pin_1) (x2)
- net at U?.14 (O5): now also J?.1 (Pin_1) (x2)
- net at U?.15 (O4): now also J?.1 (Pin_1) (x2)
- net at U?.16 (O3): now also J?.1 (Pin_1) (x2)
- net at U?.17 (O2): now also J?.1 (Pin_1) (x2)
- net at U?.18 (O1): now also J?.1 (Pin_1) (x2)
- net at U?.6 (I6): now also U?.36 (PF7)
- net at U?.7 (I7): now also U?.31 (PC6)
- net at U?.8 (I8): now also U?.32 (PC7)
- net +12V: now reaches D?.2 (A), J?.1 (Pin_1), U?.1 (VI)
- net +12V: now also R?.1
- net +5V: now reaches C?.1, C?.1, C?.1, C?.1, J?.2 (VCC), U?.14 (VCC), U?.3 (VO), U?.34 (VCC)
- net +5V: now also C?.1, C?.2, D?.2 (A), Q?.1 (S), Q?.2 (S), Q?.3 (S), R?.1, U?.6 (-)
- net MOSI: now reaches J?.4 (MOSI), U?.10 (PB2)
- net MISO: now reaches J?.1 (MISO), U?.11 (PB3)
- net RESET: now reaches J?.5 (~RST), U?.13 (~RESET)
- net RESET: now also D?.1 (K), R?.2
- net at J?.1 (VBUS), U?.2 (UVCC): now also F?.2; no longer U?.7 (VBUS)
- net at U?.33 (~HWB~/PE2): now also R?.2
- net SCK: now reaches J?.3 (SCK), U?.9 (PB1)
- net at J?.2 (D-), R?.2: now also F?.1
- net at J?.3 (D+), R?.2: now also F?.1
- new net: U?.3 (DE), U?.30 (PB6)
- new net: F?.1, U?.7 (VBUS)
- new net: C?.1, R?.1, R?.2, U?.5 (+)
- new net: Q?.4 (G), U?.7
- new net: C?.2, R?.2
- new net VBUS: Q?.5 (D), Q?.6 (D), Q?.7 (D), Q?.8 (D)
- no-connect marks 0 -> 2
Other:
- note added: "+5V AUTOSELECTOR\nUSB power on if Vin < 10v"
- note added: "12VDC"
- note added: "6 pin ICSP Connector"
- note added: "Decoupling capacitors"
- note added: "RS485 BUS"
- note added: "USB Autoreset\nTODO: risk of RESET or oRESET inverted here?"
- moved on the sheet: C?, D?, J?, R?, U?, Y?
