File: electronics/board/board.sch (KiCad schematic (older format))
At the start: 77 parts, among them J1 Screw_Terminal_01x02, J10 Conn_01x02, J11 Conn_01x02, J12 Conn_01x02, J13 Conn_01x02, J14 Conn_01x02, J15 Conn_01x02, J16 Conn_01x02, J17 Conn_01x02, J18 Conn_01x02, J19 Conn_01x02, J2 Screw_Terminal_01x02, J20 Conn_01x02, J21 Conn_01x02, J22 Conn_01x02, J23 Conn_01x02, J3 AVR-ISP-6, J4 USB_B_Micro, J5 PD1, J6 Screw_Terminal_01x02, J7 Screw_Terminal_01x02, J8 Conn_01x02, J9 Conn_01x02, Q1 IRF7404, SW1 SW_Push_Open_Dual, U1 LMV358, U2 ATmega32U4-AU, U3 NCP1117-5.0_TO252, U4 ST485EBDR, U5 ULN2803A, U6 ULN2803A, Y1 Crystal 16MHz

Commit message: Routed 1.1
Connections:
- net at U5.1 (I1): now also U2.26 (PD6); no longer U2.32 (PC7)
- net at U5.2 (I2): now also U2.27 (PD7); no longer U2.31 (PC6)
- net at U5.3 (I3): now also U2.28 (PB4); no longer U2.30 (PB6)
- net at U5.5 (I5): now also U2.30 (PB6); no longer U2.28 (PB4)
- net at U5.6 (I6): now also U2.31 (PC6); no longer U2.27 (PD7)
- net at U5.7 (I7): now also U2.32 (PC7); no longer U2.26 (PD6)
- net at U6.1 (I1): now also U2.12 (PB7); no longer U2.18 (PD0)
- net at U6.2 (I2): now also U2.18 (PD0); no longer U2.12 (PB7)
- net at U6.3 (I3): now also U2.36 (PF7); no longer U2.41 (PF0)
- net at U6.4 (I4): now also U2.37 (PF6); no longer U2.40 (PF1)
- net at U6.5 (I5): now also U2.38 (PF5); no longer U2.39 (PF4)
- net at U6.6 (I6): now also U2.39 (PF4); no longer U2.38 (PF5)
- net at U6.7 (I7): now also U2.40 (PF1); no longer U2.37 (PF6)
- net at U6.8 (I8): now also U2.41 (PF0); no longer U2.36 (PF7)
Changed lines of the file:
@@
 Wire Wire Line
 	8150 2250 8250 2250
-Wire Wire Line
-	6200 5600 8300 5600
-Wire Wire Line
-	6200 5500 8300 5500
-Wire Wire Line
-	6200 5400 8300 5400
-Wire Wire Line
-	6200 5300 8300 5300
-Wire Wire Line
-	6200 5200 8300 5200
-Wire Wire Line
-	6200 5100 8300 5100
 $Comp
 L Switch:SW_Push_Open_Dual SW1
@@
 Connection ~ 4650 1150
 Wire Wire Line
-	6200 3700 6900 3700
-Wire Wire Line
-	6900 3700 6900 3350
-Wire Wire Line
-	6900 3350 8250 3350
-Wire Wire Line
-	6200 3600 6850 3600
-Wire Wire Line
-	6850 3600 6850 3450
-Wire Wire Line
-	6850 3450 8250 3450
-Wire Wire Line
 	6200 3200 7100 3200
 Wire Wire Line
 	7100 3200 7100 3650
 Wire Wire Line
-	7100 3650 8250 3650
-Wire Wire Line
 	6200 3300 7150 3300
 Wire Wire Line
-	7150 3300 7150 3550
-Wire Wire Line
-	7150 3550 8250 3550
-Wire Wire Line
 	6200 3100 7200 3100
 Wire Wire Line
-	7200 3100 7200 3750
-Wire Wire Line
-	7200 3750 8250 3750
-Wire Wire Line
-	8250 3850 7900 3850
-Wire Wire Line
-	7900 3850 7900 4600
-Wire Wire Line
-	7900 4600 6200 4600
-Wire Wire Line
-	8250 3950 7800 3950
-Wire Wire Line
-	7800 3950 7800 4500
-Wire Wire Line
 	7800 4500 6200 4500
 Wire Wire Line
@@
 	6400 4000 6400 3900
 Wire Wire Line
-	6200 3900 6300 3900
-Wire Wire Line
-	6300 3900 6300 4650
-Wire Wire Line
-	6300 4650 8300 4650
-Wire Wire Line
-	8300 4650 8300 4900
-Wire Wire Line
 	6200 3400 6800 3400
-Wire Wire Line
-	6800 3400 6800 5000
 Wire Wire Line
 	6800 5000 8300 5000
 Connection ~ 6400 4000
+Wire Wire Line
+	7100 3650 8250 3650
+Wire Wire Line
+	6200 3700 7500 3700
+Wire Wire Line
+	7500 3700 7500 3950
+Wire Wire Line
+	7500 3950 8250 3950
+Wire Wire Line
+	7800 4500 7800 3350
+Wire Wire Line
+	7800 3350 8250 3350
+Wire Wire Line
+	6200 4600 7850 4600
+Wire Wire Line
+	7850 4600 7850 3450
+Wire Wire Line
+	7850 3450 8250 3450
+Wire Wire Line
+	7750 3600 7750 3850
+Wire Wire Line
+	7750 3850 8250 3850
+Wire Wire Line
+	6200 3600 7750 3600
+Wire Wire Line
+	7150 3300 7150 3750
+Wire Wire Line
+	7150 3750 8250 3750
+Wire Wire Line
+	7200 3100 7200 3550
+Wire Wire Line
+	7200 3550 8250 3550
+Wire Wire Line
+	6200 5600 7600 5600
+Wire Wire Line
+	7600 5600 7600 5100
+Wire Wire Line
+	7600 5100 8300 5100
+Wire Wire Line
+	6200 5100 6950 5100
+Wire Wire Line
+	6950 5100 6950 5550
+Wire Wire Line
+	6950 5550 8300 5550
+Wire Wire Line
+	8300 5550 8300 5600
+Wire Wire Line
+	6200 5500 7650 5500
+Wire Wire Line
+	7650 5500 7650 5200
+Wire Wire Line
+	7650 5200 8300 5200
+Wire Wire Line
+	6200 5400 7700 5400
+Wire Wire Line
+	7700 5400 7700 5300
+Wire Wire Line
+	7700 5300 8300 5300
+Wire Wire Line
+	6200 5200 7000 5200
+Wire Wire Line
+	7000 5200 7000 5450
+Wire Wire Line
+	7000 5450 7700 5450
+Wire Wire Line
+	7700 5450 7700 5500
+Wire Wire Line
+	7700 5500 8300 5500
+Wire Wire Line
+	6200 5300 7050 5300
+Wire Wire Line
+	7050 5300 7050 5350
+Wire Wire Line
+	7050 5350 8300 5350
+Wire Wire Line
+	8300 5350 8300 5400
+Wire Wire Line
+	6200 3900 6350 3900
+Wire Wire Line
+	6350 3900 6350 4450
+Wire Wire Line
+	6350 4450 6800 4450
+Wire Wire Line
+	6800 4450 6800 5000
+Wire Wire Line
+	6800 3400 6800 4150
+Wire Wire Line
+	6800 4150 7750 4150
+Wire Wire Line
+	7750 4150 7750 4900
+Wire Wire Line
+	7750 4900 8300 4900
 $EndSCHEMATC
